File: pinwatch/fixtures/sample_board.kicad_sch (KiCad schematic)
At the start: 1 part, among them U1 AMS1117-3.3

Commit message: feat: add automated KiCad schematic patching and ECO generation
Parts:
- U1: value AMS1117-3.3 -> AZ1117CH-3.3TRG1; MPN AMS1117-3.3 -> AZ1117CH-3.3TRG1
Changed lines of the file:
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@@
 (kicad_sch (version 20231120)
-  (symbol (lib_id "Reg:AMS1117") (property "Reference" "U1") (property "Value" "AMS1117-3.3") (property "Footprint" "SOT-223-3") (property "MPN" "AMS1117-3.3")
+  (symbol (lib_id "Reg:AMS1117") (property "Reference" "U1") (property "Value" "AZ1117CH-3.3TRG1") (property "Footprint" "SOT-223-3") (property "MPN" "AZ1117CH-3.3TRG1")
     (pin "1" (name "ADJ/GND")) (pin "2" (name "VOUT")) (pin "3" (name "VIN"))
   )
